File: Hardware/DezentraleBadge/BlinkyLogo.kicad_sch (KiCad schematic)
At the start: 50 parts, among them J101 PROG, J102 USB_C_Receptacle_USB2.0_16P, SW101 Button, U101 CH32V003AxMx

Commit message: kicad
Parts:
- J101: now fitted
Changed lines of the file:
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@@
 		(in_bom yes)
 		(on_board yes)
-		(dnp yes)
+		(dnp no)
 		(fields_autoplaced yes)
 		(property "Reference" "J101"
